File: DMR to MTM5400.kicad_pcb (KiCad board)
At the start: 2 copper layers, 101.5 x 52.5 mm, 22 parts, among them J1 MTM5400 acc.con., J2 DMR acc.conn., T1-RX1 600ohm 1:1, T2-TX1 600ohm 1:1, U1 CNY17-2, U2 CNY17-2

Commit message: Add files via upload
Parts:
- added REF**: OSHW-Logo2_7.3x6mm_SilkScreen, Symbol:OSHW-Logo2_7.3x6mm_SilkScreen, F.Cu at (165.0, 118.0)
- J2: value DMR acc.conn. -> DMR Radio acc.conn.
- renumbered T1-RX1 to T1-RX, T2-TX1 to T2-TX
Other:
- board text added: "-"
- board text added: "A_GND"
- board text added: "Ext MIC PTT"
- board text added: "GND"
- board text added: "PL/TG Det."
- board text added: "RX-A_in"
- board text added: "TX-A_out"
- board text added: "X"
