File: DMR to MTM5400.kicad_sch (KiCad schematic)
At the start: 22 parts, among them J1 MTM5400 acc.con., J2 DMR acc.conn., T1-RX1 600ohm 1:1, T2-TX1 600ohm 1:1, U1 CNY17-2, U2 CNY17-2

Commit message: Add files via upload
Other:
- note added: "Ext MIC PTT"
- note added: "PL/Talkgroup Detect"
- note removed: "GPIO"
- note removed: "PTT"
Changed lines of the file:
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@@
 		(company "Z32IT")
 	)
-	(text "PTT"
+	(text "Ext MIC PTT"
 		(exclude_from_sim no)
-		(at 55.372 75.438 0)
+		(at 56.642 74.676 0)
 		(effects
 			(font
@@
 		)
 	)
-	(text "GPIO"
+	(text "PL/Talkgroup Detect"
 		(exclude_from_sim no)
 		(at 55.626 69.088 0)
