File: V3/DMR to MTM5400 V3.kicad_pcb (KiCad board)
At the start: 2 copper layers, 101.5 x 48.2 mm, 34 parts, among them J1 MTM5400 acc.con., J2 DMR acc.conn., Q1 BC817, T1-RX 600ohm 1:1, T2-TX 600ohm 1:1, U1 CNY17-2, U2 CNY17-2, U3 L7805

Commit message: Add files via upload
Parts:
- moved C1 30.9 mm to (173.8, 98.2)
- moved C2 30.9 mm to (171.1, 123.5)
- moved C3 30.9 mm to (133.1, 91.8)
- moved C4 30.9 mm to (118.8, 96.8)
- moved C4*1 30.9 mm to (165.1, 85.8)
- moved C5 30.9 mm to (166.6, 95.6)
- moved C6 30.9 mm to (112.7, 123.2)
- moved C7 30.9 mm to (112.7, 112.2)
- moved D1 30.9 mm to (163.6, 93.6)
- moved D2 30.9 mm to (166.6, 90.3)
- moved D3 30.9 mm to (180.3, 85.8)
- moved J1 30.9 mm to (101.6, 91.2)
- moved J2 30.9 mm to (191.6, 100.0)
- moved Q1 30.9 mm to (173.0, 89.7)
- moved R1 30.9 mm to (165.1, 123.5)
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Routing:
- net GND: track 6.53 -> 0.00 mm, vias 3 -> 0
- net Net-(J2-Pin_4): track 118.9 -> 113.4 mm
Other:
- board size 101.5 x 48.2 mm -> 99.8 x 45.8 mm
